File: Relay/Schematics/Relay.brd (EAGLE design)
At the start: 100 x 80 mm, 24 parts, among them IC1 7805, Q1 16 Mhz, U1 ATMEGA328P_PDIP

Commit message: Fixed a bug on the board where the led was not wired up to a pwn pin.
Connections:
- net N$18: now also U1.17; no longer U1.14
Routing:
- net N$18: track 6.35 -> 16.8 mm
Changed lines of the file:
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@@
 <grid distance="0.05" unitdist="inch" unit="inch" style="lines" multiple="1" display="yes" altdistance="0.005" altunitdist="inch" altunit="inch"/>
 <layers>
-<layer number="1" name="Top" color="4" fill="1" visible="no" active="yes"/>
+<layer number="1" name="Top" color="4" fill="1" visible="yes" active="yes"/>
 <layer number="16" name="Bottom" color="1" fill="1" visible="yes" active="yes"/>
 <layer number="17" name="Pads" color="2" fill="1" visible="yes" active="yes"/>
 <layer number="18" name="Vias" color="2" fill="1" visible="yes" active="yes"/>
-<layer number="19" name="Unrouted" color="6" fill="1" visible="no" active="yes"/>
+<layer number="19" name="Unrouted" color="6" fill="1" visible="yes" active="yes"/>
 <layer number="20" name="Dimension" color="15" fill="1" visible="yes" active="yes"/>
-<layer number="21" name="tPlace" color="16" fill="1" visible="no" active="yes"/>
-<layer number="22" name="bPlace" color="14" fill="1" visible="no" active="yes"/>
-<layer number="23" name="tOrigins" color="15" fill="1" visible="no" active="yes"/>
-<layer number="24" name="bOrigins" color="15" fill="1" visible="no" active="yes"/>
+<layer number="21" name="tPlace" color="16" fill="1" visible="yes" active="yes"/>
+<layer number="22" name="bPlace" color="14" fill="1" visible="yes" active="yes"/>
+<layer number="23" name="tOrigins" color="15" fill="1" visible="yes" active="yes"/>
+<layer number="24" name="bOrigins" color="15" fill="1" visible="yes" active="yes"/>
 <layer number="25" name="tNames" color="7" fill="1" visible="no" active="yes"/>
 <layer number="26" name="bNames" color="7" fill="1" visible="no" active="yes"/>
@@
 <layer number="49" name="Reference" color="7" fill="1" visible="no" active="yes"/>
 <layer number="50" name="dxf" color="7" fill="1" visible="no" active="no"/>
-<layer number="51" name="tDocu" color="6" fill="1" visible="no" active="yes"/>
+<layer number="51" name="tDocu" color="6" fill="1" visible="yes" active="yes"/>
 <layer number="52" name="bDocu" color="7" fill="1" visible="no" active="yes"/>
 <layer number="53" name="tGND_GNDA" color="7" fill="9" visible="no" active="no"/>
@@
 <wire x1="86.36" y1="31.75" x2="77.47" y2="31.75" width="0.8128" layer="16"/>
 </signal>
-<signal name="N$18">
-<contactref element="R1" pad="P$1"/>
-<contactref element="U1" pad="14"/>
-<wire x1="67.31" y1="24.13" x2="60.96" y2="24.13" width="0.8128" layer="16"/>
-</signal>
 <signal name="N$19">
 <contactref element="R2" pad="P$1"/>
@@
 <via x="1.27" y="54.61" extent="1-16" drill="0.508" diameter="2.032"/>
 </signal>
+<signal name="N$18">
+<contactref element="R1" pad="P$1"/>
+<contactref element="U1" pad="17"/>
+<wire x1="67.31" y1="24.13" x2="64.77" y2="24.13" width="0.8128" layer="16"/>
+<wire x1="64.77" y1="24.13" x2="60.96" y2="27.94" width="0.8128" layer="16"/>
+<wire x1="60.96" y1="27.94" x2="55.88" y2="27.94" width="0.8128" layer="16"/>
+<wire x1="55.88" y1="27.94" x2="55.88" y2="31.75" width="0.8128" layer="16"/>
+</signal>
 </signals>
